File: old_schematic/submarine/submarine.kicad_sch (KiCad schematic)
At the start: 31 parts, among them M1 Motor_Servo, M2 Motor_Servo, M3 Motor_Servo, M4 Motor_Servo, P1 Pump Aft, P2 Pump Fwd, SW1 Power Switch, SW1 Pump Aft (P5), SW2 Manual/Auto Switch, SW2 Pump Fwd (P4)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

Commit message: 'complete' old schematic and work on new one
Parts:
- added R7, R8 (x2): 1K, symbol Device:R_US
- added U?: ms5837_depth, symbol custom_parts:ms5837_depth
Connections:
- net GND: now also R7.2, R8.2, R8.2
- net at J?.1 (Pin_1), U1.18 (5V), U3.13 (VDD): now also U?.2 (+5V)
- net at J?.3 (Pin_3), U2. (GND), U3.18 (GND): now also U?.1 (GND)
- net at U1.28 (A5), U3.23 (SCL): now also U?.3 (SCL)
- net at U1.27 (A4), U3.24 (SDA): now also U?.4 (SDA)
- net at J?.7 (Pin_7), U1.13 (12): now also R7.1
- net at J?.6 (Pin_6), U1.24 (A1): now also R8.1
- net at J?.4 (Pin_4), U1.5 (4): now also R8.1
- net at SW1.2 (B): now also J?.1 (Pin_1), SW2.2 (B), SW3.2, SW4.2, U?. (Y)
- net at U?. (Y): now also J?.3 (Pin_3); no longer J?.1 (Pin_1)
