File: electronics/v2_electronics/v2_electronics.kicad_pcb (KiCad board)
At the start: 2 copper layers, 165.1 x 101.6 mm, 48 parts, among them J1 PinHeader_1x03_P2.54mm_Vertic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, K1 Relay_SPDT_Omron-G5Q-1, K2 Relay_SPDT_Omron-G5Q-1, K3 Relay_SPDT_Omron-G5Q-1, K4 Relay_SPDT_Omron-G5Q-1, Q1 TO-92_Inline, Q2 TO-92_Inline, Q3 TO-92_Inline, Q4 TO-92_Inline, Q5 TO-92_Inline, Q6 TO-92_Inline, Q7 TO-92_Inline, Q8 TO-92_Inline, U1 metro_mini, U2 mpu6050

Commit message: start v2 pcb
Parts:
- removed 12-6V Converter: Molex_Mini-Fit_Jr_5569-08A2_2x04_P4.20mm_Horizontal, Connector_Molex:Molex_Mini-Fit_Jr_5569-08A2_2x04_P4.20mm_Horizontal
- removed 8, NC (x4): PinHeader_1x01_P2.54mm_Vertical, Connector_PinHeader_2.54mm:PinHeader_1x01_P2.54mm_Vertical
- removed Controller Battery: Molex_Mini-Fit_Jr_5569-04A2_2x02_P4.20mm_Horizontal, Connector_Molex:Molex_Mini-Fit_Jr_5569-04A2_2x02_P4.20mm_Horizontal
- removed D6, D7: LED_D5.0mm, LED_THT:LED_D5.0mm
- removed Depth Sensor: Molex_Mini-Fit_Jr_5569-04A2_2x02_P4.20mm_Horizontal, Connector_Molex:Molex_Mini-Fit_Jr_5569-04A2_2x02_P4.20mm_Horizontal
- removed Main Connector: Molex_Mini-Fit_Jr_5569-16A2_2x08_P4.20mm_Horizontal, Connector_Molex:Molex_Mini-Fit_Jr_5569-16A2_2x08_P4.20mm_Horizontal
- removed Power I/O: Molex_Mini-Fit_Jr_5569-08A2_2x04_P4.20mm_Horizontal, Connector_Molex:Molex_Mini-Fit_Jr_5569-08A2_2x04_P4.20mm_Horizontal
- removed Q7, Q8: TO-92_Inline, Package_TO_SOT_THT:TO-92_Inline
- removed R14, R15, R16: R_Axial_DIN0207_L6.3mm_D2.5mm_P10.16mm_Horizontal, Resistor_THT:R_Axial_DIN0207_L6.3mm_D2.5mm_P10.16mm_Horizontal
- added J2: Main Power, Connector_Molex:Molex_Mini-Fit_Jr_5569-08A2_2x04_P4.20mm_Horizontal, F.Cu at (258.3, 114.3)
- added J3: 12-6V Converter, Connector_Molex:Molex_Mini-Fit_Jr_5569-08A2_2x04_P4.20mm_Horizontal, F.Cu at (255.3, 71.9)
- added J4: Controller Battery Connector, Connector_Molex:Molex_Mini-Fit_Jr_5569-04A2_2x02_P4.20mm_Horizontal, F.Cu at (213.8, 71.9)
- added J5: Depth Sensor, Connector_Molex:Molex_Mini-Fit_Jr_5569-04A2_2x02_P4.20mm_Horizontal, F.Cu at (258.3, 135.1)
- added K5: T9AS1D12, custom_footprints:T9AS1D12, F.Cu at (246.1, 89.6)
- added K6: G5Q-1A 12V, Relay_THT:Relay_SPST_Omron-G5Q-1A, F.Cu at (224.8, 71.1)
- D1, D2, D3, D4: value D_DO-41_SOD81_P12.70mm_Horizontal -> 1N4007
- D5: value LED_D5.0mm -> 1N4007; footprint LED_THT:LED_D5.0mm -> Diode_THT:D_DO-41_SOD81_P10.16mm_Horizontal
- J1: value PinHeader_1x03_P2.54mm_Vertical -> Main Connector; footprint Connector_PinHeader_2.54mm:PinHeader_1x03_P2.54mm_Vertical -> Connector_Molex:Molex_Mini-Fit_Jr_5569-16A2_2x08_P4.20mm_Horizontal
- K1, K2, K3, K4: value Relay_SPDT_Omron-G5Q-1 -> G5Q-1 5V
- Q1, Q2, Q3, Q4, Q5: value TO-92_Inline -> BC547
- Q6: value TO-92_Inline -> BC557
- R1, R11, R2, R3, R4, R5, R6, R7: value R_Axial_DIN0207_L6.3mm_D2.5mm_P10.16mm_Horizontal -> 1K
- R10: value R_Axial_DIN0207_L6.3mm_D2.5mm_P15.24mm_Horizontal -> 10K; footprint Resistor_THT:R_Axial_DIN0207_L6.3mm_D2.5mm_P15.24mm_Horizontal -> Resistor_THT:R_Axial_DIN0207_L6.3mm_D2.5mm_P10.16mm_Horizontal
- R12: value R_Axial_DIN0207_L6.3mm_D2.5mm_P10.16mm_Horizontal -> 22K
- R13: value R_Axial_DIN0207_L6.3mm_D2.5mm_P10.16mm_Horizontal -> 4.7K
- R8: value R_Axial_DIN0207_L6.3mm_D2.5mm_P10.16mm_Horizontal -> 470
- R9: value R_Axial_DIN0207_L6.3mm_D2.5mm_P15.24mm_Horizontal -> 1K; footprint Resistor_THT:R_Axial_DIN0207_L6.3mm_D2.5mm_P15.24mm_Horizontal -> Resistor_THT:R_Axial_DIN0207_L6.3mm_D2.5mm_P10.16mm_Horizontal
- U1: value metro_mini -> raspberry_pi_pico; footprint custom_footprints:metro_mini -> custom_footprints:raspberry_pi_pico
- U2: value mpu6050 -> mpu6050_breakout
- moved D5 184.8 mm to (240.0, 82.5)
- moved Q1 144.1 mm to (193.0, 74.0)
- moved Q5 142.8 mm to (232.4, 128.0)
- moved Q6 141.8 mm to (238.9, 128.0)
- moved R9 137.1 mm to (238.8, 119.1), turned to 0 degrees
- moved D1 134.1 mm to (156.2, 67.6), turned to -90 degrees
- moved R5 129.6 mm to (221.0, 95.2), turned to 180 degrees
- moved R7 125.7 mm to (223.5, 97.8), turned to 0 degrees
- moved K1 125.3 mm to (161.3, 77.8)
- moved R11 124.9 mm to (238.8, 123.2), turned to 0 degrees
- moved R8 124.9 mm to (223.5, 116.6), turned to 0 degrees
- moved R6 116.6 mm to (210.8, 100.3), turned to 0 degrees
- moved R10 112.1 mm to (218.4, 110.5), turned to 0 degrees
- moved Q2 107.6 mm to (193.0, 95.2)
- moved R12 104.1 mm to (234.7, 105.4), turned to 0 degrees
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Connections:
- D1 pad 1: (no net) -> /+6V
- D1 pad 2: (no net) -> Net-(D1-Pad2)
- D2 pad 1: (no net) -> /+6V
- D2 pad 2: (no net) -> Net-(D2-Pad2)
- D3 pad 1: (no net) -> /+6V
- D3 pad 2: (no net) -> Net-(D3-Pad2)
- D4 pad 1: (no net) -> /+6V
- D4 pad 2: (no net) -> Net-(D4-Pad2)
- D5 pad 1: (no net) -> /+12V_Unswitched
- D5 pad 2: (no net) -> /MC:7
- J1 pad 1: (no net) -> /3V3
- J1 pad 2: (no net) -> /GP26
- J1 pad 3: (no net) -> /GP27
- K1 pad 1: (no net) -> Net-(D1-Pad2)
- K1 pad 2: (no net) -> /+12V
- K1 pad 3: (no net) -> /MC:13
- K1 pad 4: (no net) -> unconnected-(K1-Pad4)
- K1 pad 5: (no net) -> /+6V
- K2 pad 1: (no net) -> Net-(D2-Pad2)
- K2 pad 2: (no net) -> /+12V
- K2 pad 3: (no net) -> /MC:14
- K2 pad 4: (no net) -> unconnected-(K2-Pad4)
- K2 pad 5: (no net) -> /+6V
- K3 pad 1: (no net) -> Net-(D3-Pad2)
- K3 pad 2: (no net) -> /+12V
- K3 pad 3: (no net) -> /MC:15
- K3 pad 4: (no net) -> unconnected-(K3-Pad4)
- K3 pad 5: (no net) -> /+6V
- K4 pad 1: (no net) -> Net-(D4-Pad2)
- K4 pad 2: (no net) -> /+12V
- K4 pad 3: (no net) -> /MC:16
- K4 pad 4: (no net) -> unconnected-(K4-Pad4)
- K4 pad 5: (no net) -> /+6V
- Q1 pad 1: (no net) -> Net-(D1-Pad2)
- Q1 pad 2: (no net) -> Net-(Q1-Pad2)
- Q1 pad 3: (no net) -> GND
- Q2 pad 1: (no net) -> Net-(D2-Pad2)
- Q2 pad 2: (no net) -> Net-(Q2-Pad2)
- Q2 pad 3: (no net) -> GND
- Q3 pad 1: (no net) -> Net-(D3-Pad2)
- Q3 pad 2: (no net) -> Net-(Q3-Pad2)
- Q3 pad 3: (no net) -> GND
- Q4 pad 1: (no net) -> Net-(D4-Pad2)
- Q4 pad 2: (no net) -> Net-(Q4-Pad2)
- Q4 pad 3: (no net) -> GND
- Q5 pad 1: (no net) -> Net-(Q5-Pad1)
- Q5 pad 2: (no net) -> Net-(Q5-Pad2)
- Q5 pad 3: (no net) -> GND
- Q6 pad 1: (no net) -> Net-(Q6-Pad1)
- Q6 pad 2: (no net) -> /External LED
- Q6 pad 3: (no net) -> /+6V
- R1 pad 1: (no net) -> Net-(Q1-Pad2)
- R1 pad 2: (no net) -> /GP2
- R10 pad 1: (no net) -> /+6V
- R10 pad 2: (no net) -> Net-(Q5-Pad1)
- R11 pad 1: (no net) -> /GP9
- R11 pad 2: (no net) -> Net-(Q5-Pad2)
- R12 pad 1: (no net) -> /GP28
- R12 pad 2: (no net) -> /+12V
- R13 pad 1: (no net) -> GND
- R13 pad 2: (no net) -> /GP28
- R2 pad 1: (no net) -> Net-(Q2-Pad2)
- R2 pad 2: (no net) -> /GP3
- R3 pad 1: (no net) -> Net-(Q3-Pad2)
- R3 pad 2: (no net) -> /GP4
- R4 pad 1: (no net) -> Net-(Q4-Pad2)
- R4 pad 2: (no net) -> /GP5
- R5 pad 1: (no net) -> GND
- R5 pad 2: (no net) -> /GP6
- R6 pad 1: (no net) -> GND
- R6 pad 2: (no net) -> /GP7
- R7 pad 1: (no net) -> GND
- R7 pad 2: (no net) -> /Blow Button
- R8 pad 1: (no net) -> /External LED
- R8 pad 2: (no net) -> Net-(J2-Pad2)
- R9 pad 1: (no net) -> Net-(Q5-Pad1)
- R9 pad 2: (no net) -> Net-(Q6-Pad1)
- U1 pad 1: (no net) -> /GP0
- U1 pad 10: (no net) -> /GP7
- U1 pad 11: (no net) -> /Blow Button
- U1 pad 12: (no net) -> /GP9
- U1 pad 13: (no net) -> GND
- U1 pad 14: (no net) -> /GP10
- U1 pad 15: (no net) -> /GP11
- U1 pad 16: (no net) -> /GP12
- U1 pad 17: (no net) -> /GP13
- U1 pad 18: (no net) -> GND
- U1 pad 19: (no net) -> /GP14
- U1 pad 2: (no net) -> /GP1
- U1 pad 20: (no net) -> /GP15
- U1 pad 21: (no net) -> /GP16
- U1 pad 22: (no net) -> /GP17
- U1 pad 23: (no net) -> GND
- U1 pad 24: (no net) -> /GP18
- U1 pad 25: (no net) -> /GP19
- U1 pad 26: (no net) -> /GP20
- U1 pad 27: (no net) -> /GP21
- U1 pad 3: (no net) -> GND
- U1 pad 4: (no net) -> /GP2
- U1 pad 5: (no net) -> /GP3
- U1 pad 6: (no net) -> /GP4
- U1 pad 7: (no net) -> /GP5
- U1 pad 8: (no net) -> GND
- U1 pad 9: (no net) -> /GP6
- U2 pad 1: (no net) -> /3V3
- U2 pad 2: (no net) -> GND
- U2 pad 3: (no net) -> /GP1
- U2 pad 4: (no net) -> /GP0
- U2 pad 5: (no net) -> unconnected-(U2-Pad5)
- U2 pad 6: (no net) -> unconnected-(U2-Pad6)
- U2 pad 7: (no net) -> unconnected-(U2-Pad7)
- U2 pad 8: (no net) -> unconnected-(U2-Pad8)
Routing:
- net (no net): track 4416.7 -> 0.00 mm, vias 21 -> 0
- net /+6V: track 0.00 -> 166.1 mm
- net /+12V: track 0.00 -> 139.1 mm
- net GND: track 0.00 -> 89.1 mm
- net /MC:13: track 0.00 -> 77.6 mm
- net Net-(D3-Pad2): track 0.00 -> 71.4 mm
- net Net-(D4-Pad2): track 0.00 -> 65.9 mm
- net /MC:14: track 0.00 -> 50.2 mm
- net /MC:15: track 0.00 -> 47.1 mm
- net Net-(D1-Pad2): track 0.00 -> 42.3 mm
- net Net-(D2-Pad2): track 0.00 -> 42.0 mm
- net /+12V_Unswitched: track 0.00 -> 34.3 mm
- net /MC:16: track 0.00 -> 18.3 mm
- net /MC:7: track 0.00 -> 8.75 mm
Other:
- board outline removed
- board text removed: "+12V"
- board text removed: "+5V"
- board text removed: "+6V"
- board text removed: "1"
- board text removed: "10"
- board text removed: "11"
- board text removed: "12"
- board text removed: "13"
- board text removed: "14"
- board text removed: "15"
- board text removed: "16"
- board text removed: "2"
- board text removed: "3"
- board text removed: "4"
- board text removed: "5"
- board text removed: "6"
- board text removed: "7"
- board text removed: "8"
- board text removed: "9"
- board text removed: "Button/Switch Pulldown Resistors"
- board text removed: "C B E"
- board text removed: "External LED"
- board text removed: "GND"
- board text removed: "LED Resistors"
- board text removed: "LED Transistor Resistors"
- board text removed: "MPU6050"
- board text removed: "Relay Transistor Resistors"
- board text removed: "SCL"
- board text removed: "SDA"
- board text removed: "Status LEDs"
- board text removed: "Vbat"

Commit message: do most of the work on v2 pcb
Parts:
- moved R7 85.0 mm to (139.1, 107.3), turned to 180 degrees
- moved R5 82.1 mm to (139.1, 101.0)
- moved R6 71.9 mm to (139.1, 104.1), turned to 180 degrees
- moved U2 52.7 mm to (223.3, 141.5), turned to 90 degrees
- moved R4 44.8 mm to (200.4, 89.9)
- moved R3 40.8 mm to (204.0, 89.9)
- moved R2 37.8 mm to (207.5, 89.9)
- moved R1 36.1 mm to (211.1, 89.9)
- moved R11 19.8 mm to (223.5, 135.9)
- moved R10 19.8 mm to (232.4, 124.5), turned to 180 degrees
- moved R9 16.6 mm to (222.2, 120.7)
- moved Q6 15.8 mm to (231.1, 114.3)
- moved D5 14.8 mm to (225.3, 83.8)
- moved R12 14.1 mm to (222.8, 98.0), turned to 90 degrees
- moved J2 12.8 mm to (245.6, 115.6)
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Connections:
- Q6 pad 1: Net-(Q6-Pad1) -> /External LED
- Q6 pad 2: /External LED -> Net-(R9-Pad2)
- R9 pad 2: Net-(Q6-Pad1) -> Net-(R9-Pad2)
Routing:
- net GND: track 89.1 -> 451.8 mm
- net /MC:7: track 8.75 -> 200.4 mm
- net /+6V: track 166.1 -> 335.5 mm
- net /3V3: track 0.00 -> 127.5 mm
- net /GP6: track 0.00 -> 106.5 mm
- net /GP7: track 0.00 -> 94.1 mm, vias 0 -> 1
- net /GP1: track 0.00 -> 88.9 mm
- net /+12V: track 139.1 -> 221.2 mm
- net /GP27: track 0.00 -> 81.9 mm
- net /VSYS: track 0.00 -> 78.6 mm, vias 0 -> 1
- net /Blow Button: track 0.00 -> 73.2 mm, vias 0 -> 1
- net /GP26: track 0.00 -> 72.7 mm
- net /GP9: track 0.00 -> 54.2 mm
- net /GP10: track 0.00 -> 51.6 mm
- net /GP0: track 0.00 -> 50.8 mm
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Other:
- board outline added: 143.5 x 88.9 mm

Commit message: maybe do some work on the v2 pcb
Parts:
- added REF**: MountingHole_3.2mm_M3_Pad_Via, MountingHole:MountingHole_3.2mm_M3_Pad_Via, F.Cu at (156.2, 138.4)
- moved Q2 3.81 mm to (193.0, 91.4)
- moved Q4 3.81 mm to (186.7, 91.4)
Routing:
- net Net-(D2-Pad2): track 42.0 -> 44.3 mm
- net Net-(Q2-Pad2): track 16.2 -> 17.5 mm
- net Net-(D4-Pad2): track 65.9 -> 65.4 mm

Commit message: 'finish' pcbv2, waiting for logo...
Parts:
- added J6: PinHeader_1x02_P2.54mm_Vertical, Connector_PinHeader_2.54mm:PinHeader_1x02_P2.54mm_Vertical, F.Cu at (158.1, 134.6)
- added J7: PinHeader_1x08_P2.54mm_Vertical, Connector_PinHeader_2.54mm:PinHeader_1x08_P2.54mm_Vertical, F.Cu at (165.1, 139.7)
- added J8: PinHeader_1x03_P2.54mm_Vertical, Connector_PinHeader_2.54mm:PinHeader_1x03_P2.54mm_Vertical, F.Cu at (197.5, 142.9)
- added REF**: MountingHole_3.2mm_M3_Pad_Via, MountingHole:MountingHole_3.2mm_M3_Pad_Via, F.Cu at (216.5, 135.3)
- added REF**: MountingHole_3.2mm_M3_Pad_Via, MountingHole:MountingHole_3.2mm_M3_Pad_Via, F.Cu at (122.0, 62.3)
- added REF**: MountingHole_3.2mm_M3_Pad_Via, MountingHole:MountingHole_3.2mm_M3_Pad_Via, F.Cu at (217.5, 79.3)
- added REF**: MountingHole_3.2mm_M3_Pad_Via, MountingHole:MountingHole_3.2mm_M3_Pad_Via, F.Cu at (189.5, 101.8)
- REF**: value MountingHole_3.2mm_M3_Pad_Via -> locked
- moved REF** 3.97 mm to (152.5, 139.8)
Routing:
- net /GP14: track 0.00 -> 24.1 mm
- net /GP15: track 0.00 -> 20.5 mm
- net /VBUS: track 0.00 -> 15.1 mm
- net /3V3_EN: track 0.00 -> 13.0 mm
- net /ADC_VREF: track 0.00 -> 12.0 mm
- net /RUN: track 0.00 -> 9.58 mm
- net /GP22: track 0.00 -> 9.58 mm
- net /GP17: track 0.00 -> 9.58 mm
- net /GP16: track 0.00 -> 9.54 mm
- net /GP20: track 0.00 -> 8.53 mm
- net /GP21: track 0.00 -> 8.53 mm
- net /GP19: track 0.00 -> 8.53 mm
- net /GP18: track 0.00 -> 8.53 mm
- net /MC:7: track 200.4 -> 194.5 mm
- net /GP27: track 81.9 -> 87.3 mm
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
Commit message: electronics final final?
Other:
- board text added: "Electronics Team: Ethan Clarke, Evan Vandergoot"
- board text added: "Sussex Tech Engineering - Umptysquatch X - ISR 17 - 2023"
Changed lines of the file:
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@@
       (drillshape 0)
       (scaleselection 1)
-      (outputdirectory "C:/Users/asdf/Desktop/plot-output/")
+      (outputdirectory "/home/asdf/plot_output")
     )
   )
@@
     (pad "" np_thru_hole circle (at 0 -7.3 90) (size 3 3) (drill 3) (layers *.Cu *.Mask))
     (pad "" np_thru_hole circle (at 29.4 -7.3 90) (size 3 3) (drill 3) (layers *.Cu *.Mask))
-    (pad "1" thru_hole roundrect (at 0 0 90) (size 2.7 3.7) (drill 1.8) (layers *.Cu *.Mask) (roundrect_rratio 0.092593)
+    (pad "1" thru_hole roundrect (at 0 0 90) (size 2.7 3.7) (drill 1.8) (layers *.Cu *.Mask) (roundrect_rratio 0.09259296296)
       (net 30 "/3V3") (pinfunction "Pin_1") (pintype "passive"))
     (pad "2" thru_hole oval (at 4.2 0 90) (size 2.7 3.7) (drill 1.8) (layers *.Cu *.Mask)
@@
     (pad "" np_thru_hole circle (at 0 -7.3) (size 3 3) (drill 3) (layers *.Cu *.Mask))
     (pad "" np_thru_hole circle (at 12.6 -7.3) (size 3 3) (drill 3) (layers *.Cu *.Mask))
-    (pad "1" thru_hole roundrect (at 0 0) (size 2.7 3.7) (drill 1.8) (layers *.Cu *.Mask) (roundrect_rratio 0.092593)
+    (pad "1" thru_hole roundrect (at 0 0) (size 2.7 3.7) (drill 1.8) (layers *.Cu *.Mask) (roundrect_rratio 0.09259296296)
       (net 47 "/+6V") (pinfunction "Pin_1") (pintype "passive"))
     (pad "2" thru_hole oval (at 4.2 0) (size 2.7 3.7) (drill 1.8) (layers *.Cu *.Mask)
@@
     (descr "Through hole straight pin header, 1x02, 2.54mm pitch, single row")
     (tags "Through hole pin header THT 1x02 2.54mm single row")
-    (attr through_hole)
+    (attr through_hole board_only)
     (fp_text reference "J6" (at 0 -2.33) (layer "F.SilkS")
       (effects (font (size 1 1) (thickness 0.15)))
@@
     (descr "Mounting Hole 3.2mm, M3")
     (tags "mounting hole 3.2mm m3")
-    (attr exclude_from_pos_files exclude_from_bom)
+    (attr board_only exclude_from_pos_files exclude_from_bom)
     (fp_text reference "REF**" (at 0 -4.2) (layer "F.SilkS") hide
       (effects (font (size 1 1) (thickness 0.15)))
@@
     (descr "Mounting Hole 3.2mm, M3")
     (tags "mounting hole 3.2mm m3")
-    (attr exclude_from_pos_files exclude_from_bom)
+    (attr board_only exclude_from_pos_files exclude_from_bom)
     (fp_text reference "REF**" (at 0 -4.2) (layer "F.SilkS") hide
       (effects (font (size 1 1) (thickness 0.15)))
@@
     (descr "Mounting Hole 3.2mm, M3")
     (tags "mounting hole 3.2mm m3")
-    (attr exclude_from_pos_files exclude_from_bom)
+    (attr board_only exclude_from_pos_files exclude_from_bom)
     (fp_text reference "REF**" (at 0 -4.2) (layer "F.SilkS") hide
       (effects (font (size 1 1) (thickness 0.15)))
@@
     (fp_circle (center 0 0) (end 3.2 0) (layer "Cmts.User") (width 0.15) (fill none))
     (fp_circle (center 0 0) (end 3.45 0) (layer "F.CrtYd") (width 0.05) (fill none))
-    (pad "1" thru_hole circle locked (at 0 0) (size 6.4 6.4) (drill 3.2) (layers *.Cu *.Mask))
+    (pad "1" thru_hole circle locked (at -2.4 0) (size 0.8 0.8) (drill 0.5) (layers *.Cu *.Mask))
     (pad "1" thru_hole circle locked (at 0 2.4) (size 0.8 0.8) (drill 0.5) (layers *.Cu *.Mask))
     (pad "1" thru_hole circle locked (at 2.4 0) (size 0.8 0.8) (drill 0.5) (layers *.Cu *.Mask))
     (pad "1" thru_hole circle locked (at 0 -2.4) (size 0.8 0.8) (drill 0.5) (layers *.Cu *.Mask))
     (pad "1" thru_hole circle locked (at -1.697056 -1.697056) (size 0.8 0.8) (drill 0.5) (layers *.Cu *.Mask))
+    (pad "1" thru_hole circle locked (at 0 0) (size 6.4 6.4) (drill 3.2) (layers *.Cu *.Mask))
+    (pad "1" thru_hole circle locked (at 1.697056 1.697056) (size 0.8 0.8) (drill 0.5) (layers *.Cu *.Mask))
+    (pad "1" thru_hole circle locked (at 1.697056 -1.697056) (size 0.8 0.8) (drill 0.5) (layers *.Cu *.Mask))
     (pad "1" thru_hole circle locked (at -1.697056 1.697056) (size 0.8 0.8) (drill 0.5) (layers *.Cu *.Mask))
-    (pad "1" thru_hole circle locked (at -2.4 0) (size 0.8 0.8) (drill 0.5) (layers *.Cu *.Mask))
-    (pad "1" thru_hole circle locked (at 1.697056 -1.697056) (size 0.8 0.8) (drill 0.5) (layers *.Cu *.Mask))
-    (pad "1" thru_hole circle locked (at 1.697056 1.697056) (size 0.8 0.8) (drill 0.5) (layers *.Cu *.Mask))
   )
   (footprint "Package_TO_SOT_THT:TO-92_Inline" (layer "F.Cu")
@@
     (fp_line (start -2.7 -1.1) (end 6.9 -1.1) (layer "F.Fab") (width 0.1))
     (pad "" np_thru_hole circle (at 2.1 -7.3 270) (size 3 3) (drill 3) (layers *.Cu *.Mask))
-    (pad "1" thru_hole roundrect (at 0 0 270) (size 2.7 3.7) (drill 1.8) (layers *.Cu *.Mask) (roundrect_rratio 0.092593)
+    (pad "1" thru_hole roundrect (at 0 0 270) (size 2.7 3.7) (drill 1.8) (layers *.Cu *.Mask) (roundrect_rratio 0.09259296296)
       (net 3 "GND") (pinfunction "Pin_1") (pintype "passive"))
     (pad "2" thru_hole oval (at 4.2 0 270) (size 2.7 3.7) (drill 1.8) (layers *.Cu *.Mask)
@@
     (pad "" np_thru_hole circle (at 12.6 -7.3 270) (size 3 3) (drill 3) (layers *.Cu *.Mask))
     (pad "" np_thru_hole circle (at 0 -7.3 270) (size 3 3) (drill 3) (layers *.Cu *.Mask))
-    (pad "1" thru_hole roundrect (at 0 0 270) (size 2.7 3.7) (drill 1.8) (layers *.Cu *.Mask) (roundrect_rratio 0.092593)
+    (pad "1" thru_hole roundrect (at 0 0 270) (size 2.7 3.7) (drill 1.8) (layers *.Cu *.Mask) (roundrect_rratio 0.09259296296)
       (net 39 "/+12V_Unswitched") (pinfunction "Pin_1") (pintype "passive"))
     (pad "2" thru_hole oval (at 4.2 0 270) (size 2.7 3.7) (drill 1.8) (layers *.Cu *.Mask)
@@
     (descr "Through hole straight pin header, 1x03, 2.54mm pitch, single row")
     (tags "Through hole pin header THT 1x03 2.54mm single row")
-    (attr through_hole)
+    (attr through_hole board_only)
     (fp_text reference "J8" (at 0 -2.33 90) (layer "F.SilkS")
       (effects (font (size 1 1) (thickness 0.15)))
@@
     (descr "Mounting Hole 3.2mm, M3")
     (tags "mounting hole 3.2mm m3")
-    (attr exclude_from_pos_files exclude_from_bom)
+    (attr board_only exclude_from_pos_files exclude_from_bom)
     (fp_text reference "REF**" (at 0 -4.2) (layer "F.SilkS") hide
       (effects (font (size 1 1) (thickness 0.15)))
@@
     (descr "Mounting Hole 3.2mm, M3")
     (tags "mounting hole 3.2mm m3")
-    (attr exclude_from_pos_files exclude_from_bom)
+    (attr board_only exclude_from_pos_files exclude_from_bom)
     (fp_text reference "REF**" (at 0 -4.2) (layer "F.SilkS") hide
       (effects (font (size 1 1) (thickness 0.15)))
@@
     (fp_line (start 6.9 -13.9) (end -2.7 -13.9) (layer "F.Fab") (width 0.1))
     (pad "" np_thru_hole circle (at 2.1 -7.3) (size 3 3) (drill 3) (layers *.Cu *.Mask))
-    (pad "1" thru_hole roundrect (at 0 0) (size 2.7 3.7) (drill 1.8) (layers *.Cu *.Mask) (roundrect_rratio 0.092593)
+    (pad "1" thru_hole roundrect (at 0 0) (size 2.7 3.7) (drill 1.8) (layers *.Cu *.Mask) (roundrect_rratio 0.09259296296)
       (net 48 "Net-(J4-Pad1)") (pinfunction "Pin_1") (pintype "passive"))
     (pad "2" thru_hole oval (at 4.2 0) (size 2.7 3.7) (drill 1.8) (layers *.Cu *.Mask)
@@
     (descr "Through hole straight pin header, 1x08, 2.54mm pitch, single row")
     (tags "Through hole pin header THT 1x08 2.54mm single row")
-    (attr through_hole)
+    (attr through_hole board_only)
     (fp_text reference "J7" (at 0 -2.33 90) (layer "F.SilkS")
       (effects (font (size 1 1) (thickness 0.15)))
@@
   )
   (gr_rect locked (start 117.475 57.785) (end 260.985 146.685) (layer "Edge.Cuts") (width 0.1) (fill none))
+  (gr_text "Electronics Team: Ethan Clarke, Evan Vandergoot" (at 127 64.135) (layer "F.SilkS")
+    (effects (font (size 1.5 1.5) (thickness 0.3)) (justify left))
+  )
+  (gr_text "Sussex Tech Engineering - Umptysquatch X - ISR 17 - 2023" (at 127 60.96) (layer "F.SilkS")
+    (effects (font (size 1.5 1.5) (thickness 0.3)) (justify left))
+  )
   (segment (start 228.092 134.747) (end 228.092 136.667) (width 0.5) (layer "F.Cu") (net 1))
   (segment (start 229.855 138.43) (end 228.092 136.667) (width 0.5) (layer "F.Cu") (net 1))
@@
   (segment (start 128.905 117.33) (end 132.815 121.24) (width 0.5) (layer "B.Cu") (net 10))
   (segment (start 128.905 107.315) (end 128.905 110.49) (width 0.5) (layer "B.Cu") (net 10))
+  (segment (start 223.52 135.89) (end 214.63 127) (width 0.5) (layer "F.Cu") (net 11))
   (segment (start 182.938 120.708) (end 182.938 113.412) (width 0.5) (layer "F.Cu") (net 11))
-  (segment (start 223.52 135.255) (end 215.265 127) (width 0.5) (layer "F.Cu") (net 11))
-  (segment (start 223.52 135.89) (end 223.52 135.255) (width 0.5) (layer "F.Cu") (net 11))
-  (segment (start 215.265 127) (end 189.23 127) (width 0.5) (layer "F.Cu") (net 11))
+  (segment (start 214.63 127) (end 189.23 127) (width 0.5) (layer "F.Cu") (net 11))
   (segment (start 189.23 127) (end 182.938 120.708) (width 0.5) (layer "F.Cu") (net 11))
   (segment (start 142.24 142.24) (end 138.315 142.24) (width 1) (layer "F.Cu") (net 12))
