File: electronics/v2_electronics/v2_electronics.kicad_sch (KiCad schematic)
At the start: 30 parts, among them J1 Main Connector, J2 Main Power, J3 12-6V Converter, J4 Battery Connector, J5 Depth Sensor, K1 G5Q-1, K2 G5Q-1, K3 G5Q-1, K4 G5Q-1, Q1 BC547, Q2 BC547, Q3 BC547, Q4 BC547, Q8 BC547, U1 raspberry_pi_pico, U2 mpu6050_breakout

Commit message: more work v2 electronics
Parts:
- U2: footprint (none) -> custom_footprints:mpu6050
Connections:
- net MC:1 is gone; now on net 3V3: J1.1 (Pin_1)
- net MC:10 is gone; now on net GP11: J1.10 (Pin_10)
- net MC:11 is gone; now on net GP12: J1.11 (Pin_11)
- net MC:12 is gone; now on net GP13: J1.12 (Pin_12)
- net MC:2 is gone; now on net GP26: J1.2 (Pin_2)
- net MC:3 is gone; now on net GP27: J1.3 (Pin_3)
- net MC:4 is gone; now on net GP6: J1.4 (Pin_4), R5.2
- net MC:5 is gone; now on net GP7: J1.5 (Pin_5), R6.2
- net MC:6 is gone; now on net Blow Button: J1.6 (Pin_6), R7.2
- net MC:7 is gone; now on net GP9: J1.7 (Pin_7), R8.2
- net MC:9 is gone; now on net GP10: J1.9 (Pin_9)
- net External LED Power renamed External LED
- net GP8 renamed Blow Button
Other:
- note added: "Main Connector - Controller Connections"
- note added: "NC"
- note added: "change resistor for external led"
- note added: "check servo numbers!!"
- note added: "figure out power switch!!"
- note added: "some sorta voltage divider for main voltage here"
- moved on the sheet: R5, R6, R7, R8

Commit message: more pcb v2 work:
Parts:
- removed R8: 1K, Resistor_THT:R_Axial_DIN0207_L6.3mm_D2.5mm_P10.16mm_Horizontal, symbol Device:R_US
- added K5: T9AS1D12-12, TE_1-1393210-3, symbol custom_parts:T9AS1D12
- added Q9: BC557, symbol Device:Q_PNP_BCE
- added R17, R18: 1K, Resistor_THT:R_Axial_DIN0207_L6.3mm_D2.5mm_P10.16mm_Horizontal, symbol Device:R_US
- added R19: 22K, Resistor_THT:R_Axial_DIN0207_L6.3mm_D2.5mm_P10.16mm_Horizontal, symbol Device:R_US
- added R20: 4.7K, Resistor_THT:R_Axial_DIN0207_L6.3mm_D2.5mm_P10.16mm_Horizontal, symbol Device:R_US
- J4: value Battery Connector -> Controller Battery Connector
Connections:
- net External LED Control is gone; now on net +6V: R16.1
- net +12V: now also R19.2
- net +6V: now also Q9.3 (E); no longer Q8.1 (C)
- net External LED: now also Q9.2 (C); no longer Q8.3 (E)
- net GND: now also Q8.3 (E), R20.1
- net GP14: now also R18.1
- net GP28: now also R19.1, R20.2
- net GP9: now also K5.A1
- net at R16.2: now also Q8.1 (C), R17.1; no longer Q8.2 (B)
- new net: Q8.2 (B), R18.2
- new net: Q9.1 (B), R17.2
- new net: K5.A2, K5.NO
- no-connect marks 0 -> 1
Other:
- note added: "12V battery voltage divider"
- note added: "High-side driver for external LED"
- note removed: "NC"
- note removed: "change resistor for external led"
- note removed: "some sorta voltage divider for main voltage here"
- moved on the sheet: D1, D2, D3, D4, J1, J2, J3, J4, J5, K1, K2, K3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

Commit message: more work on schematic v2
Parts:
- added D5: 1N4007, Diode_THT:D_DO-41_SOD81_P10.16mm_Horizontal, symbol Diode:1N4007
- K5: value T9AS1D12-12 -> T9AS1D12; footprint TE_1-1393210-3 -> custom_footprints:T9AS1D12
- Q9: footprint (none) -> Package_TO_SOT_THT:TO-92_Inline
Connections:
- net +12V: now also K5.C; no longer J2.1 (Pin_1), J2.5 (Pin_5), K1.2, K2.2, K3.2, K4.2, R19.2
- net GP14: no longer R18.1
- net GP9: now also R18.1; no longer J1.7 (Pin_7), K5.A1
- net at K5.A2, K5.NO: now also J2.1 (Pin_1), J2.5 (Pin_5), K1.2, K2.2, K3.2, K4.2, R19.2, D5.1 (K)
- new net MC:7: D5.2 (A), J1.7 (Pin_7), K5.A1
- no-connect marks 1 -> 6
Other:
- note added: "Button pulldown resistors"
- note removed: "figure out power switch!!"
- moved on the sheet: J2, R15, R5, R6, R7

Commit message: more work on v2 schematic:
Connections:
- net VSYS: no longer J4.1 (Pin_1), J4.2 (Pin_2)
- new net: J4.1 (Pin_1), J4.2 (Pin_2)
Other:
- note added: "pick a 12v lower current relay"
- note added: "pick a smaller relay (>=15a)"
- moved on the sheet: J4
Changed lines of the file:
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@@
 (kicad_sch (version 20211123) (generator eeschema)
   (paper "A")
+  (bus_alias "ControllerPins" (members "GP0" "GP1" "GND" "GP2" "GP3" "GP4" "GP5" "GP6" "GP7" "GP8" "GP9" "GP10" "GP11" "GP12" "GP13" "GP14" "GP15" "GP16" "GP17" "GP18" "GP19" "GP20" "GP21" "GP22" "GP26" "GP27" "GP28" "ADC_VREF" "3V3" "3V3_EN" "VSYS" "VBUS"))
   (bus_alias "MainConnector" (members "MC:1" "MC:2" "MC:3" "MC:4" "MC:5" "MC:6" "MC:7" "MC:8" "MC:9" "MC:10" "MC:11" "MC:12" "MC:13" "MC:14" "MC:15" "MC:16"))
-  (bus_alias "ControllerPins" (members "GP0" "GP1" "GND" "GP2" "GP3" "GP4" "GP5" "GP6" "GP7" "GP8" "GP9" "GP10" "GP11" "GP12" "GP13" "GP14" "GP15" "GP16" "GP17" "GP18" "GP19" "GP20" "GP21" "GP22" "GP26" "GP27" "GP28" "ADC_VREF" "3V3" "3V3_EN" "VSYS" "VBUS"))
   (junction (at 226.06 44.45) (diameter 0) (color 0 0 0 0)
   )
@@
   (junction (at 154.94 16.51) (diameter 0) (color 0 0 0 0)
   )
-  (junction (at 157.48 149.86) (diameter 0) (color 0 0 0 0)
+  (junction (at 198.12 151.13) (diameter 0) (color 0 0 0 0)
   )
   (junction (at 204.47 107.95) (diameter 0) (color 0 0 0 0)
@@
   )
   (junction (at 254 64.77) (diameter 0) (color 0 0 0 0)
-  )
-  (junction (at 151.13 143.51) (diameter 0) (color 0 0 0 0)
   )
   (junction (at 220.98 120.65) (diameter 0) (color 0 0 0 0)
@@
     (stroke (width 0) (type default) (color 0 0 0 0))
   )
-  (wire (pts (xy 144.78 143.51) (xy 151.13 143.51))
-    (stroke (width 0) (type default) (color 0 0 0 0))
-  )
   (bus (pts (xy 135.89 107.95) (xy 135.89 110.49))
     (stroke (width 0) (type default) (color 0 0 0 0))
@@
     (stroke (width 0) (type default) (color 0 0 0 0))
   )
-  (wire (pts (xy 163.83 142.24) (xy 163.83 144.78))
+  (wire (pts (xy 204.47 143.51) (xy 204.47 146.05))
     (stroke (width 0) (type default) (color 0 0 0 0))
   )
@@
     (stroke (width 0) (type default) (color 0 0 0 0))
   )
-  (wire (pts (xy 151.13 147.32) (xy 151.13 149.86))
+  (wire (pts (xy 191.77 148.59) (xy 191.77 151.13))
     (stroke (width 0) (type default) (color 0 0 0 0))
   )
@@
     (stroke (width 0) (type default) (color 0 0 0 0))
   )
-  (wire (pts (xy 151.13 143.51) (xy 151.13 144.78))
-    (stroke (width 0) (type default) (color 0 0 0 0))
-  )
   (wire (pts (xy 156.21 91.44) (xy 171.45 91.44))
     (stroke (width 0) (type default) (color 0 0 0 0))
@@
     (stroke (width 0) (type default) (color 0 0 0 0))
   )
-  (wire (pts (xy 151.13 142.24) (xy 151.13 143.51))
+  (wire (pts (xy 191.77 143.51) (xy 191.77 146.05))
     (stroke (width 0) (type default) (color 0 0 0 0))
   )
@@
     (stroke (width 0) (type default) (color 0 0 0 0))
   )
-  (wire (pts (xy 163.83 149.86) (xy 163.83 147.32))
+  (wire (pts (xy 204.47 151.13) (xy 204.47 148.59))
     (stroke (width 0) (type default) (color 0 0 0 0))
   )
@@
     (stroke (width 0) (type default) (color 0 0 0 0))
   )
-  (wire (pts (xy 157.48 149.86) (xy 163.83 149.86))
+  (wire (pts (xy 198.12 151.13) (xy 204.47 151.13))
     (stroke (width 0) (type default) (color 0 0 0 0))
   )
@@
     (stroke (width 0) (type default) (color 0 0 0 0))
   )
-  (wire (pts (xy 151.13 149.86) (xy 157.48 149.86))
+  (wire (pts (xy 191.77 151.13) (xy 198.12 151.13))
     (stroke (width 0) (type default) (color 0 0 0 0))
   )
@@
     (stroke (width 0) (type default) (color 0 0 0 0))
   )
-  (wire (pts (xy 163.83 142.24) (xy 151.13 142.24))
+  (wire (pts (xy 204.47 143.51) (xy 191.77 143.51))
     (stroke (width 0) (type default) (color 0 0 0 0))
   )
@@
     (stroke (width 0) (type default) (color 0 0 0 0))
   )
+  (wire (pts (xy 144.78 143.51) (xy 165.1 143.51))
+    (stroke (width 0) (type default) (color 0 0 0 0))
+  )
   (wire (pts (xy 110.49 92.71) (xy 133.35 92.71))
     (stroke (width 0) (type default) (color 0 0 0 0))
@@
     (stroke (width 0) (type default) (color 0 0 0 0))
   )
+  (text "pick a smaller relay (>=15a)" (at 232.41 60.96 0)
+    (effects (font (size 1.27 1.27)) (justify left bottom))
+  )
   (text "12V battery voltage divider" (at 162.56 82.55 0)
     (effects (font (size 1.27 1.27)) (justify left bottom))
@@
   )
   (text "High-side driver for external LED" (at 191.77 125.73 0)
+    (effects (font (size 1.27 1.27)) (justify left bottom))
+  )
+  (text "pick a 12v lower current relay" (at 160.02 149.86 0)
     (effects (font (size 1.27 1.27)) (justify left bottom))
   )
@@
     (pin "1")
   )
-  (symbol (lib_name "GND_2") (lib_id "power:GND") (at 157.48 149.86 0) (mirror y) (unit 1)
+  (symbol (lib_name "GND_2") (lib_id "power:GND") (at 198.12 151.13 0) (mirror y) (unit 1)
     (in_bom yes) (on_board yes) (fields_autoplaced)
-    (property "Reference" "#PWR0102" (id 0) (at 157.48 156.21 0)
-      (effects (font (size 1.27 1.27)) hide)
-    )
-    (property "Value" "GND" (id 1) (at 157.48 154.94 0))
-    (property "Footprint" "" (id 2) (at 157.48 149.86 0)
-      (effects (font (size 1.27 1.27)) hide)
-    )
-    (property "Datasheet" "" (id 3) (at 157.48 149.86 0)
+    (property "Reference" "#PWR0102" (id 0) (at 198.12 157.48 0)
+      (effects (font (size 1.27 1.27)) hide)
+    )
+    (property "Value" "GND" (id 1) (at 198.12 156.21 0))
+    (property "Footprint" "" (id 2) (at 198.12 151.13 0)
+      (effects (font (size 1.27 1.27)) hide)
+    )
+    (property "Datasheet" "" (id 3) (at 198.12 151.13 0)
       (effects (font (size 1.27 1.27)) hide)
     )
@@
     (pin "3")
   )
-  (symbol (lib_id "Connector_Generic:Conn_02x02_Odd_Even") (at 158.75 144.78 0) (mirror y) (unit 1)
+  (symbol (lib_id "Connector_Generic:Conn_02x02_Odd_Even") (at 199.39 146.05 0) (mirror y) (unit 1)
     (in_bom yes) (on_board yes)
-    (property "Reference" "J4" (id 0) (at 157.48 137.16 0))
-    (property "Value" "Controller Battery Connector" (id 1) (at 157.48 139.7 0))
-    (property "Footprint" "Connector_Molex:Molex_Mini-Fit_Jr_5569-04A2_2x02_P4.20mm_Horizontal" (id 2) (at 158.75 144.78 0)
-      (effects (font (size 1.27 1.27)) hide)
-    )
-    (property "Datasheet" "~" (id 3) (at 158.75 144.78 0)
-      (effects (font (size 1.27 1.27)) hide)
-    )
+    (property "Reference" "J4" (id 0) (at 198.12 138.43 0))
+    (property "Value" "Controller Battery Connector" (id 1) (at 198.12 140.97 0))
+    (property "Footprint" "Connector_Molex:Molex_Mini-Fit_Jr_5569-04A2_2x02_P4.20mm_Horizontal" (id 2) (at 199.39 146.05 0)
+      (effects (font (size 1.27 1.27)) hide)
+    )
+    (property "Datasheet" "~" (id 3) (at 199.39 146.05 0)
+      (effects (font (size 1.27 1.27)) hide)
+    )

Commit message: start v2 pcb
Parts:
- added K6: G5Q-1A 12V, Relay_THT:Relay_SPST_Omron-G5Q-1A, symbol Relay:G5Q-1A
- K1, K2, K3, K4: value G5Q-1 -> G5Q-1 5V
- renumbered Q8 to Q5, Q9 to Q6, R16 to R10, R18 to R11, R19 to R12, R20 to R13, R15 to R8, R17 to R9
Connections:
- net +12V: now also K1.2, K2.2, K3.2, K4.2, R12.2
- net MC:7: now also K6.5
- net VSYS: now also K6.3
- net +12V_Unswitched: now reaches D5.1 (K), J2.1 (Pin_1), J2.5 (Pin_5), K5.A2, K5.NO
- net +12V_Unswitched: now also K6.1; no longer K1.2, K2.2, K3.2, K4.2, R12.2
- net at J4.1 (Pin_1), J4.2 (Pin_2): now also K6.2
Other:
- note removed: "pick a 12v lower current relay"
- note removed: "pick a smaller relay (>=15a)"
- moved on the sheet: J4

Commit message: do most of the work on v2 pcb
Parts:
- removed Q6: BC557, Package_TO_SOT_THT:TO-92_Inline, symbol Device:Q_PNP_BCE
- added Q6: BC557, Package_TO_SOT_THT:TO-92_Inline, symbol Device:Q_PNP_CBE
Connections:
- net +6V: now also Q6.3 (E)
- net External LED: now also Q6.1 (C)
- net at R9.2: now also Q6.2 (B)
Changed lines of the file:
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@@
 (kicad_sch (version 20211123) (generator eeschema)
   (paper "A")
+  (bus_alias "ControllerPins" (members "GP0" "GP1" "GND" "GP2" "GP3" "GP4" "GP5" "GP6" "GP7" "GP8" "GP9" "GP10" "GP11" "GP12" "GP13" "GP14" "GP15" "GP16" "GP17" "GP18" "GP19" "GP20" "GP21" "GP22" "GP26" "GP27" "GP28" "ADC_VREF" "3V3" "3V3_EN" "VSYS" "VBUS"))
   (bus_alias "MainConnector" (members "MC:1" "MC:2" "MC:3" "MC:4" "MC:5" "MC:6" "MC:7" "MC:8" "MC:9" "MC:10" "MC:11" "MC:12" "MC:13" "MC:14" "MC:15" "MC:16"))
-  (bus_alias "ControllerPins" (members "GP0" "GP1" "GND" "GP2" "GP3" "GP4" "GP5" "GP6" "GP7" "GP8" "GP9" "GP10" "GP11" "GP12" "GP13" "GP14" "GP15" "GP16" "GP17" "GP18" "GP19" "GP20" "GP21" "GP22" "GP26" "GP27" "GP28" "ADC_VREF" "3V3" "3V3_EN" "VSYS" "VBUS"))
   (junction (at 226.06 44.45) (diameter 0) (color 0 0 0 0)
   )
@@
     (pin "4")
   )
-  (symbol (lib_id "Device:Q_PNP_BCE") (at 218.44 107.95 0) (unit 1)
-    (in_bom yes) (on_board yes) (fields_autoplaced)
-    (property "Reference" "Q6" (id 0) (at 223.52 106.6799 0)
-      (effects (font (size 1.27 1.27)) (justify left))
-    )
-    (property "Value" "BC557" (id 1) (at 223.52 109.2199 0)
-      (effects (font (size 1.27 1.27)) (justify left))
-    )
-    (property "Footprint" "Package_TO_SOT_THT:TO-92_Inline" (id 2) (at 223.52 105.41 0)
-      (effects (font (size 1.27 1.27)) hide)
-    )
-    (property "Datasheet" "~" (id 3) (at 218.44 107.95 0)
-      (effects (font (size 1.27 1.27)) hide)
-    )
-    (pin "1")
-    (pin "2")
-    (pin "3")
-  )
   (symbol (lib_id "Relay:G5Q-1") (at 77.47 30.48 0) (unit 1)
     (in_bom yes) (on_board yes) (fields_autoplaced)
@@
     (pin "7")
     (pin "8")
+  )
+  (symbol (lib_id "Device:Q_PNP_CBE") (at 218.44 107.95 0) (unit 1)
+    (in_bom yes) (on_board yes) (fields_autoplaced)
+    (property "Reference" "Q6" (id 0) (at 223.52 106.6799 0)
+      (effects (font (size 1.27 1.27)) (justify left))
+    )
+    (property "Value" "BC557" (id 1) (at 223.52 109.2199 0)
+      (effects (font (size 1.27 1.27)) (justify left))
+    )
+    (property "Footprint" "Package_TO_SOT_THT:TO-92_Inline" (id 2) (at 223.52 105.41 0)
+      (effects (font (size 1.27 1.27)) hide)
+    )
+    (property "Datasheet" "~" (id 3) (at 218.44 107.95 0)
+      (effects (font (size 1.27 1.27)) hide)
+    )
+    (pin "1")
+    (pin "2")
+    (pin "3")
   )
   (symbol (lib_id "Relay:G5Q-1") (at 160.02 30.48 0) (unit 1)
@@
       (reference "Q5") (unit 1) (value "BC547") (footprint "Package_TO_SOT_THT:TO-92_Inline")
     )
-    (path "/a55468bc-3c04-4b7e-8b55-45b4eeb83798"
+    (path "/d0bf7106-c7d7-4ee5-a8b9-00191a8266cf"
       (reference "Q6") (unit 1) (value "BC557") (footprint "Package_TO_SOT_THT:TO-92_Inline")
     )

Commit message: electronics final final?
Other:
- title: (none) -> Umptysquatch X Electronics
Changed lines of the file:
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@@
 (kicad_sch (version 20211123) (generator eeschema)
   (paper "A")
+  (title_block
+    (title "Umptysquatch X Electronics")
+    (rev "2")
+  )
+  (bus_alias "MainConnector" (members "MC:1" "MC:2" "MC:3" "MC:4" "MC:5" "MC:6" "MC:7" "MC:8" "MC:9" "MC:10" "MC:11" "MC:12" "MC:13" "MC:14" "MC:15" "MC:16"))
   (bus_alias "ControllerPins" (members "GP0" "GP1" "GND" "GP2" "GP3" "GP4" "GP5" "GP6" "GP7" "GP8" "GP9" "GP10" "GP11" "GP12" "GP13" "GP14" "GP15" "GP16" "GP17" "GP18" "GP19" "GP20" "GP21" "GP22" "GP26" "GP27" "GP28" "ADC_VREF" "3V3" "3V3_EN" "VSYS" "VBUS"))
-  (bus_alias "MainConnector" (members "MC:1" "MC:2" "MC:3" "MC:4" "MC:5" "MC:6" "MC:7" "MC:8" "MC:9" "MC:10" "MC:11" "MC:12" "MC:13" "MC:14" "MC:15" "MC:16"))
   (junction (at 226.06 44.45) (diameter 0) (color 0 0 0 0)
   )
