File: electronics/v2_electronics/v2_electronics.kicad_sch (KiCad schematic)
At the start: 37 parts, among them J1 Main Connector, J2 Main Power, J3 12-6V Converter, J4 Controller Battery Connector, J5 Depth Sensor, K1 G5Q-1 5V, K2 G5Q-1 5V, K3 G5Q-1 5V, K4 G5Q-1 5V, K5 T9AS1D12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

Commit message: modify pcb and schematic sheets for export for design report
Other:
- note removed: "check servo numbers!!"
- company: (none) -> Sussex Tech Engineering
Changed lines of the file:
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@@
   (title_block
     (title "Umptysquatch X Electronics")
+    (date "4/9/2023")
     (rev "2")
+    (company "Sussex Tech Engineering")
   )
   (bus_alias "ControllerPins" (members "GP0" "GP1" "GND" "GP2" "GP3" "GP4" "GP5" "GP6" "GP7" "GP8" "GP9" "GP10" "GP11" "GP12" "GP13" "GP14" "GP15" "GP16" "GP17" "GP18" "GP19" "GP20" "GP21" "GP22" "GP26" "GP27" "GP28" "ADC_VREF" "3V3" "3V3_EN" "VSYS" "VBUS"))
@@
     (effects (font (size 1.27 1.27)) (justify left bottom))
   )
-  (text "check servo numbers!!" (at 101.6 121.92 0)
-    (effects (font (size 1.27 1.27)) (justify left bottom))
-  )
