File: electronics/new_electronics/new_electronics.kicad_sch (KiCad schematic)
At the start: 47 parts, among them J1 Conn_01x05_Female, J2 5-Pin Power Connector, J3 Conn_01x16_Female, J4 16-Pin Connector, K1 G5Q-1, K2 G5Q-1, K3 G5Q-1, K4 G5Q-1, M1 Motor_Servo, M2 Motor_Servo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

Commit message: modify pcb and schematic sheets for export for design report
Other:
- company: (none) -> Sussex Tech Engineering
- title: (none) -> Umptysquatch X Electronics
